Commit message: Add ETH reference flow and camera/IBVS integration updates

File: src/ur5e_ts_ibvs_description/urdf/ur5e_ibvs_setup.urdf.xacro (robot description, xacro)
@@ -35,4 +35,5 @@
   <xacro:include filename="$(find ur5e_ts_ibvs_description)/urdf/robotiq_85_gripper.urdf.xacro"/>
   <xacro:include filename="$(find ur5e_ts_ibvs_description)/urdf/realsense_d435.urdf.xacro"/>
+  <xacro:include filename="$(find ur5e_ts_ibvs_description)/urdf/overview_camera.urdf.xacro"/>
   <xacro:include filename="$(find ur5e_ts_ibvs_description)/urdf/objects.urdf.xacro"/>
   <!-- ======== Properties ======== -->
@@ -91,4 +92,25 @@
     <origin xyz="${wrist_length} 0 0" rpy="0 0 0"/>
   </xacro:robotiq_85_gripper>
+  <!-- ======== Green marker on the gripper (eye-to-hand) ======== -->
+  <!-- Bright green plate the fixed overview camera tracks as the controlled
+       feature set. Visual-only (no collision) so planning is unaffected.
+       Same size/placement as the ROS1 setup. -->
+  <link name="ee_marker_link">
+    <visual>
+      <origin xyz="0 0 0" rpy="0 0 0"/>
+      <geometry>
+        <box size="0.05 0.05 0.005"/>
+      </geometry>
+      <material name="MarkerGreen">
+        <color rgba="0.0 1.0 0.0 1.0"/>
+      </material>
+    </visual>
+  </link>
+  <joint name="ee_marker_joint" type="fixed">
+    <parent link="gripper_base_link"/>
+    <child link="ee_marker_link"/>
+    <!-- Sits on top of the gripper base, facing up -->
+    <origin xyz="0.0 0.0 0.04" rpy="0 0 0"/>
+  </joint>
   <!-- ======== Table ======== -->
   <xacro:mytable/>
@@ -98,4 +120,11 @@
     <origin xyz="0.7 0.0 ${table_height}" rpy="0 0 0"/>
   </joint>
+  <!-- ======== Fixed overview camera (eye-to-hand) ======== -->
+  <!-- Same mounting as ROS1: close to the workspace so the TS scheduling
+       range (Z in [0.25, 0.85] m) is well exercised. Looks down/back at the
+       cube and the gripper marker. -->
+  <xacro:overview_camera parent="table">
+    <origin xyz="0.55 0.0 0.60" rpy="${pi} ${4.0*pi/5.0} 0"/>
+  </xacro:overview_camera>
   <!-- ======== Red Target Cube (on table) ======== -->
   <xacro:red_target/>

Commit message: Update robot setup and runtime scripts

File: src/ur5e_ts_ibvs_description/urdf/ur5e_ibvs_setup.urdf.xacro (robot description, xacro)
@@ -113,4 +113,29 @@
     <origin xyz="0.0 0.0 0.04" rpy="0 0 0"/>
   </joint>
+  <!-- ======== Cable frames (SOFA Cosserat coupling) ======== -->
+  <!-- Physical clamp point of the cable between the fingertips. The SOFA
+       cable base is driven by base_link -> cable_grasp_frame. x points out
+       of the fingers = initial cable direction. -->
+  <link name="cable_grasp_frame"/>
+  <joint name="cable_grasp_joint" type="fixed">
+    <parent link="gripper_base_link"/>
+    <child link="cable_grasp_frame"/>
+    <origin xyz="0.14 0 0" rpy="0 0 0"/>
+  </joint>
+  <!-- Table fixture clamping the far cable end (planar shaping setup).
+       +x = initial cable direction (world +y); cable free end lands near
+       world (0.45, 0.35), inside the arm workspace. Small visible clamp. -->
+  <link name="cable_fixture_frame">
+    <visual>
+      <origin xyz="0 0 0" rpy="0 0 0"/>
+      <geometry><box size="0.03 0.03 0.05"/></geometry>
+      <material name="FixtureYellow"><color rgba="0.9 0.8 0.1 1.0"/></material>
+    </visual>
+  </link>
+  <joint name="cable_fixture_joint" type="fixed">
+    <parent link="table"/>
+    <child link="cable_fixture_frame"/>
+    <origin xyz="-0.25 -0.35 0.03" rpy="0 0 ${pi/2}"/>
+  </joint>
   <!-- ======== Table ======== -->
   <xacro:mytable/>
@@ -132,6 +157,6 @@
     <parent link="table"/>
     <child link="red_target"/>
-    <!-- World x=0.4 (matches ROS1 spawn -x 0.4), on the table surface -->
-    <origin xyz="-0.3 0.0 ${0.025 + 0.025}" rpy="0 0 0"/>
+    <!-- Moved to the far table corner, clear of the cable workspace -->
+    <origin xyz="-0.3 -0.7 ${0.025 + 0.025}" rpy="0 0 0"/>
   </joint>
   <!-- ======== gz-sim ros2_control plugin ======== -->
